File: design/BatteryLevelIndicator/BatteryLevelIndicator.kicad_pcb (KiCad board)
At the start: 2 copper layers, 60.3 x 9.8 mm, 14 parts, among them J1 Conn_01x10_MountingPin, SW3 power

Commit message: adjustement and gerber files
Parts:
- C1: value C -> 100nF; footprint Capacitor_SMD:C_0805_2012Metric -> Capacitor_SMD:C_0603_1608Metric_Pad1.08x0.95mm_HandSolder
- R11, R12, R8: value R -> 1kΩ; footprint Resistor_SMD:R_0805_2012Metric -> Resistor_SMD:R_0402_1005Metric_Pad0.72x0.64mm_HandSolder
Routing:
- net power: track 31.5 -> 32.0 mm
